File: craftwalk.kicad_pcb (KiCad board)
At the start: 2 copper layers, 137.3 x 98.9 mm, 44 parts, among them J1 LED, SW1 RESET_SW, U1 ProMicro

Commit message: rev 1.2
- add LED support
- change libs to submodule
- refactor
Parts:
- removed J1: LED, kbd:StripLED_rev
- added L1: YS-SK6812MINI, craftwalk:YS-SK6812, F.Cu at (80.0, 75.4)
- added L10: YS-SK6812MINI, craftwalk:YS-SK6812-underglow, F.Cu at (91.5, 67.4)
- added L11: YS-SK6812MINI, craftwalk:YS-SK6812-underglow, F.Cu at (110.6, 62.7)
- added L12: YS-SK6812MINI, craftwalk:YS-SK6812-underglow, F.Cu at (129.6, 67.8)
- added L13: YS-SK6812MINI, craftwalk:YS-SK6812-underglow, F.Cu at (70.8, 89.5)
- added L14: YS-SK6812MINI, craftwalk:YS-SK6812-underglow, F.Cu at (91.5, 86.6)
- added L15: YS-SK6812MINI, craftwalk:YS-SK6812-underglow, F.Cu at (110.6, 82.1)
- added L16: YS-SK6812MINI, craftwalk:YS-SK6812-underglow, F.Cu at (129.6, 86.9)
- added L17: YS-SK6812MINI, craftwalk:YS-SK6812-underglow, F.Cu at (148.7, 82.0)
- added L18: YS-SK6812MINI, craftwalk:YS-SK6812-underglow, F.Cu at (164.9, 106.0)
- added L19: YS-SK6812MINI, craftwalk:YS-SK6812-underglow, F.Cu at (182.3, 114.3)
- added L2: YS-SK6812MINI, craftwalk:YS-SK6812, F.Cu at (110.8, 48.5)
- added L3: YS-SK6812MINI, craftwalk:YS-SK6812, F.Cu at (115.0, 91.1)
- added L4: YS-SK6812MINI, craftwalk:YS-SK6812, F.Cu at (143.3, 91.7)
- added L5: YS-SK6812MINI, craftwalk:YS-SK6812, F.Cu at (164.9, 117.0)
- added L6: YS-SK6812MINI, craftwalk:YS-SK6812-underglow, F.Cu at (91.5, 48.7)
- added L7: YS-SK6812MINI, craftwalk:YS-SK6812-underglow, F.Cu at (110.6, 44.1)
- added L8: YS-SK6812MINI, craftwalk:YS-SK6812-underglow, F.Cu at (129.7, 48.5)
- added L9: YS-SK6812MINI, craftwalk:YS-SK6812-underglow, F.Cu at (66.6, 70.4)
- SW1: moved to B.Cu
- moved D8 2.45 mm to (79.5, 89.4)
Routing:
- net GND: track 131.1 -> 631.9 mm, vias 2 -> 36
- net VCC: track 126.6 -> 499.4 mm, vias 2 -> 34
- net LED: track 142.8 -> 58.9 mm
- net Net-(L1-Pad4): track 0.00 -> 59.9 mm, vias 0 -> 4
- net Net-(L1-Pad2): track 0.00 -> 46.5 mm, vias 0 -> 4
- net Net-(L18-Pad4): track 0.00 -> 43.9 mm, vias 0 -> 2
- net Net-(L4-Pad2): track 0.00 -> 34.4 mm, vias 0 -> 2
- net Net-(L17-Pad4): track 0.00 -> 34.1 mm, vias 0 -> 4
- net Net-(L10-Pad4): track 0.00 -> 28.7 mm, vias 0 -> 2
- net Net-(L13-Pad2): track 0.00 -> 28.4 mm, vias 0 -> 2
- net Net-(L7-Pad4): track 0.00 -> 28.4 mm, vias 0 -> 4
- net Net-(L12-Pad2): track 0.00 -> 28.3 mm, vias 0 -> 2
- net Net-(L3-Pad2): track 0.00 -> 23.8 mm
- net Net-(L19-Pad4): track 0.00 -> 19.9 mm, vias 0 -> 2
- net Net-(L15-Pad4): track 0.00 -> 19.2 mm, vias 0 -> 2
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Other:
- outline, holes or cut-outs redrawn
- board text added: "craftWalk PCB rev.1.2"
- board text removed: "craftWalk PCB rev.1.0"
